File: LED_ring/LED_ring.kicad_sch (KiCad schematic)
At the start: 15 parts, among them U1 BC546

Commit message: Changed values on resistors
Parts:
- removed U1: BC546, Mechatronics:TO-92_ONS, symbol Mechatronics:BC546
- R1, R2, R3: value 180 -> 100
- renumbered 12V_in1 to 12V_in1_ENABLE, ENABLE1 to GND
Connections:
- net at CR3.1, CR6.1, CR9.1: now also GND.1 (Pin_1)
Other:
- moved on the sheet: GND
Changed lines of the file:
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@@
-	(wire
-		(pts
-			(xy 252.73 110.49) (xy 259.08 110.49)
-		)
-		(stroke
-			(width 0)
-			(type default)
-		)
-	)
 	(wire
 		(pts
@@
 	(wire
 		(pts
-			(xy 259.08 110.49) (xy 259.08 115.57)
-		)
-		(stroke
-			(width 0)
-			(type default)
-		)
-	)
-	(wire
-		(pts
 			(xy 142.24 59.69) (xy 161.29 59.69)
 		)
@@
 	(wire
 		(pts
-			(xy 232.41 116.84) (xy 247.65 116.84)
+			(xy 269.875 59.69) (xy 250.19 59.69)
 		)
 		(stroke
@@
 		(pts
 			(xy 250.19 82.55) (xy 250.19 83.82)
-		)
-		(stroke
-			(width 0)
-			(type default)
-		)
-	)
-	(wire
-		(pts
-			(xy 247.65 116.84) (xy 247.65 110.49)
 		)
 		(stroke
@@
 			)
 		)
-		(property "Value" "180"
+		(property "Value" "100"
 			(at 165.1 78.74 0)
 			(effects
@@
 			)
 		)
-		(property "Value" "180"
+		(property "Value" "100"
 			(at 165.1 31.75 0)
 			(effects
@@
 			)
 		)
-		(property "Value" "180"
+		(property "Value" "100"
 			(at 165.1 55.88 0)
 			(effects
@@
 		(dnp no)
 		(fields_autoplaced yes)
-		(property "Reference" "12V_in1"
+		(property "Reference" "12V_in1_ENABLE"
 			(at 123.825 54.61 0)
 			(effects
@@
 			(project ""
 				(path "/c7b4129d-c051-430e-b09b-c9fd6f723e94"
-					(reference "12V_in1")
+					(reference "12V_in1_ENABLE")
 					(unit 1)
 				)
@@
 	)
 	(symbol
-		(lib_id "power:GND")
-		(at 259.08 115.57 0)
-		(unit 1)
-		(exclude_from_sim no)
-		(in_bom yes)
-		(on_board yes)
-		(dnp no)
-		(fields_autoplaced yes)
-		(property "Reference" "#PWR01"
-			(at 259.08 121.92 0)
-			(effects
-				(font
-					(size 1.27 1.27)
-				)
-				(hide yes)
-			)
-		)
-		(property "Value" "GND"
-			(at 259.08 120.65 0)
-			(effects
-				(font
-					(size 1.27 1.27)
-				)
-			)
-		)
-		(property "Footprint" ""
-			(at 259.08 115.57 0)
-			(effects
-				(font
-					(size 1.27 1.27)
-				)
-				(hide yes)
-			)
-		)
-		(property "Datasheet" ""
-			(at 259.08 115.57 0)
-			(effects
-				(font
-					(size 1.27 1.27)
-				)
-				(hide yes)
-			)
-		)
-		(property "Description" "Power symbol creates a global label with name \"GND\" , ground"
-			(at 259.08 115.57 0)
-			(effects
-				(font
-					(size 1.27 1.27)
-				)
-				(hide yes)
-			)
-		)
-		(pin "1"
-		)
-		(instances
-			(project ""
-				(path "/c7b4129d-c051-430e-b09b-c9fd6f723e94"
-					(reference "#PWR01")
-					(unit 1)
-				)
-			)
-		)
-	)
-	(symbol
-		(lib_id "Mechatronics:BC546")
-		(at 251.46 68.58 270)
-		(unit 1)
-		(exclude_from_sim no)
-		(in_bom yes)
-		(on_board yes)
-		(dnp no)
-		(fields_autoplaced yes)
-		(property "Reference" "U1"
-			(at 256.54 95.8849 90)
-			(effects
-				(font
-					(size 1.524 1.524)
-				)
-				(justify left)
-			)
-		)
-		(property "Value" "BC546"
-			(at 256.54 98.4249 90)
-			(effects
-				(font
-					(size 1.524 1.524)
-				)
-				(justify left)
-			)
-		)
-		(property "Footprint" "Mechatronics:TO-92_ONS"
-			(at 243.078 96.774 0)
-			(effects
-				(font
-					(size 1.27 1.27)
-					(italic yes)
-				)
-				(hide yes)
-			)
-		)
-		(property "Datasheet" "BC546"
-			(at 240.538 94.488 0)
-			(effects
-				(font
-					(size 1.27 1.27)
-					(italic yes)
-				)
-				(hide yes)
-			)
-		)
-		(property "Description" ""
-			(at 251.46 68.58 0)
-			(effects
-				(font
-					(size 1.27 1.27)
-				)
-				(hide yes)
-			)
-		)
-		(pin "2"
-		)
-		(pin "3"
-		)
-		(pin "1"
-		)
-		(instances
-			(project ""
-				(path "/c7b4129d-c051-430e-b09b-c9fd6f723e94"
-					(reference "U1")
-					(unit 1)
-				)
-			)
-		)
-	)
-	(symbol
 		(lib_id "Mechatronics:TLLG4401")
 		(at 177.8 35.56 0)
@@
 	(symbol
 		(lib_id "Connector:Conn_01x01_Pin")
-		(at 227.33 116.84 0)
-		(unit 1)
-		(exclude_from_sim no)
-		(in_bom yes)
-		(on_board yes)
-		(dnp no)
-		(fields_autoplaced yes)
-		(property "Reference" "ENABLE1"
-			(at 227.965 111.76 0)
+		(at 274.955 59.69 0)
+		(mirror y)
+		(unit 1)
+		(exclude_from_sim no)
+		(in_bom yes)
+		(on_board yes)
+		(dnp no)
+		(fields_autoplaced yes)
+		(property "Reference" "GND"
+			(at 274.32 54.61 0)
 			(effects
 				(font
@@
 		)
 		(property "Value" "Conn_01x01_Pin"
-			(at 227.965 114.3 0)
+			(at 274.32 57.15 0)
 			(effects
 				(font
@@
 		)
 		(property "Footprint" "Connector_PinHeader_2.54mm:PinHeader_1x01_P2.54mm_Vertical"
-			(at 227.33 116.84 0)
+			(at 274.955 59.69 0)
 			(effects
 				(font
@@
 		)
 		(property "Datasheet" "~"
-			(at 227.33 116.84 0)
+			(at 274.955 59.69 0)
 			(effects
 				(font
@@
 		)
 		(property "Description" "Generic connector, single row, 01x01, script generated"
-			(at 227.33 119.38 0)
-			(effects
-				(font
-					(size 1.27 1.27)
-				)
-				(hide yes)
-			)
-		)
-		(pin "1"
-		)
-		(instances
-			(project ""
-				(path "/c7b4129d-c051-430e-b09b-c9fd6f723e94"
-					(reference "ENABLE1")
-					(unit 1)
-				)
+			(at 274.955 62.23 0)
+			(effects
+				(font
+					(size 1.27 1.27)
+				)
+				(hide yes)
+			)
+		)
+		(pin "1"
+		)
+		(instances
+			(project ""
+				(path "/c7b4129d-c051-430e-b09b-c9fd6f723e94"
+					(reference "GND")
+					(unit 1)
+				)

Commit message: Modified to fit with new spec
Parts:
- added GND1a1, GND1b1, GND2a1, GND2b1, GND3a1, GND3b1, J1a1, J1b1, J2a1, J2b1, J3a1, J3b1: Conn_01x01_Pin, Connector_PinHeader_2.54mm:PinHeader_1x01_P2.54mm_Vertical, symbol Connector:Conn_01x01_Pin
- CR1: footprint Mechatronics:TLL_Series_VIS -> LED_ring:TLL_Series_VIS
- CR2, CR3, CR4, CR5, CR6, CR7, CR8, CR9: footprint TLL_Series_VIS -> LED_ring:TLL_Series_VIS
- renumbered 12V_in1_ENABLE to 12V_in1_ENABLE1, GND to GND1
Connections:
- net at R3.1: now also J3a1.1 (Pin_1); no longer CR7.2
- net at R1.1: now also J1a1.1 (Pin_1); no longer CR1.2
- net at R2.1: now also J2a1.1 (Pin_1); no longer CR4.2
- new net: CR6.1, GND2a1.1 (Pin_1)
- new net: CR3.1, GND1a1.1 (Pin_1)
- new net: CR4.2, J2b1.1 (Pin_1)
- new net: CR9.1, GND3a1.1 (Pin_1)
- new net: GND1.1 (Pin_1), GND1b1.1 (Pin_1), GND2b1.1 (Pin_1), GND3b1.1 (Pin_1)
- new net: CR7.2, J3b1.1 (Pin_1)
- new net: CR1.2, J1b1.1 (Pin_1)
Other:
- moved on the sheet: 12V_in1_ENABLE1, CR1, CR2, CR3, CR4, CR5, CR6, CR7, CR8, CR9, GND1, R1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

Commit message: Finalized PCB design
Parts:
- R1, R2, R3: footprint Resistor_THT:R_Axial_DIN0207_L6.3mm_D2.5mm_P2.54mm_Vertical -> Resistor_THT:R_Axial_DIN0204_L3.6mm_D1.6mm_P5.08mm_Horizontal
Changed lines of the file:
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@@
 			)
 		)
-		(property "Footprint" "Resistor_THT:R_Axial_DIN0207_L6.3mm_D2.5mm_P2.54mm_Vertical"
+		(property "Footprint" "Resistor_THT:R_Axial_DIN0204_L3.6mm_D1.6mm_P5.08mm_Horizontal"
 			(at 105.41 80.772 0)
 			(effects
@@
 			)
 		)
-		(property "Footprint" "Resistor_THT:R_Axial_DIN0207_L6.3mm_D2.5mm_P2.54mm_Vertical"
+		(property "Footprint" "Resistor_THT:R_Axial_DIN0204_L3.6mm_D1.6mm_P5.08mm_Horizontal"
 			(at 105.41 33.782 0)
 			(effects
@@
 			)
 		)
-		(property "Footprint" "Resistor_THT:R_Axial_DIN0207_L6.3mm_D2.5mm_P2.54mm_Vertical"
+		(property "Footprint" "Resistor_THT:R_Axial_DIN0204_L3.6mm_D1.6mm_P5.08mm_Horizontal"
 			(at 105.41 57.912 0)
 			(effects
