File: Power_regulator/Power_regulator.kicad_pcb (KiCad board)
At the start: 2 copper layers, 116.2 x 137.5 mm, 30 parts, among them J0 54-00166, J1 Conn_01x02_Pin, J1_1 Conn_01x01_Pin, J1_GND1 Conn_01x02_Pin, J1_GND_1 Conn_01x01_Pin, J2 Conn_01x01_Pin, J2_1 Conn_01x01_Pin, J2_GND1 Conn_01x01_Pin, J2_GND_1 Conn_01x01_Pin, J3 Conn_01x15_Pin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

Commit message: Finalized design for power regulator
Parts:
- R1, R2, R3, R4, R5: footprint Resistor_THT:R_Axial_DIN0207_L6.3mm_D2.5mm_P5.08mm_Vertical -> Resistor_THT:R_Axial_DIN0204_L3.6mm_D1.6mm_P7.62mm_Horizontal
- moved F2 246.1 mm to (48.6, 150.3)
- moved F3 237.4 mm to (48.7, 139.3)
- moved F4 230.0 mm to (48.6, 128.5)
- moved J0 225.8 mm to (49.7, 94.4), turned to -90 degrees
- moved F5 222.7 mm to (49.1, 117.2)
- moved F6 217.5 mm to (48.9, 106.8)
- moved R5 216.4 mm to (86.1, 139.0)
- moved R3 213.4 mm to (85.6, 123.6)
- moved R2 211.8 mm to (85.5, 116.0)
- moved J5_GND1 210.5 mm to (67.6, 91.4), turned to 90 degrees
- moved R1 210.3 mm to (85.5, 108.4)
- moved R4 208.7 mm to (93.0, 131.4), turned to 180 degrees
- moved Q5 207.0 mm to (68.5, 148.5)
- moved J4_GND1 205.7 mm to (68.1, 66.6), turned to 90 degrees
- moved F1 205.6 mm to (50.8, 58.3)
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Connections:
- net Net-(J5-Pin_1) renamed +12V
Routing:
- net +12V: track 0.00 -> 54.9 mm
- net GND: track 0.00 -> 47.0 mm
- net Net-(J3-Pin_14): track 0.00 -> 31.9 mm
- net Net-(J3-Pin_11): track 0.00 -> 30.9 mm
- net Net-(J3-Pin_2): track 0.00 -> 30.5 mm
- net Net-(J3-Pin_8): track 0.00 -> 29.8 mm
- net Net-(J3-Pin_5): track 0.00 -> 28.8 mm
- net Net-(J1-Pin_1): track 0.00 -> 24.3 mm
- net Net-(J1_GND1-Pin_1): track 0.00 -> 19.9 mm
- net Net-(Q5-B): track 0.00 -> 19.2 mm
- net Net-(Q4-B): track 0.00 -> 17.5 mm
- net Net-(Q1-B): track 0.00 -> 17.2 mm
- net Net-(Q3-B): track 0.00 -> 16.7 mm
- net Net-(Q2-B): track 0.00 -> 15.6 mm
- net Net-(Q5-C): track 0.00 -> 15.6 mm
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- added copper zone on F.Cu, net +12V
- added copper zone on B.Cu, net GND
Other:
- board size 116.2 x 137.5 mm -> 108.7 x 113 mm

Commit message: PCB done
Parts:
- moved J5 1.70 mm to (67.6, 80.7)
- moved J4_GND1 0.51 mm to (68.0, 67.1)
Routing:
- net +12V: track 54.9 -> 54.1 mm
Changed lines of the file:
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@@
 	(footprint "Connector_PinHeader_2.54mm:PinHeader_1x01_P2.54mm_Vertical"
 		(layer "F.Cu")
-		(at 67.6656 79.0194 90)
+		(at 67.564 80.7212 90)
 		(descr "Through hole straight pin header, 1x01, 2.54mm pitch, single row")
 		(tags "Through hole pin header THT 1x01 2.54mm single row")
@@
 	(footprint "Connector_PinHeader_2.54mm:PinHeader_1x01_P2.54mm_Vertical"
 		(layer "F.Cu")
-		(at 68.072 66.6242 90)
+		(at 67.9958 67.1322 90)
 		(descr "Through hole straight pin header, 1x01, 2.54mm pitch, single row")
 		(tags "Through hole pin header THT 1x01 2.54mm single row")
@@
 	)
 	(segment
+		(start 63.2222 80.8482)
+		(end 58.2176 85.8528)
+		(width 1)
+		(layer "F.Cu")
+		(net 1)
+	)
+	(segment
 		(start 50.83175 58.3184)
 		(end 50.83175 78.46695)
@@
 	)
 	(segment
-		(start 67.6656 79.0194)
-		(end 65.051 79.0194)
+		(start 67.437 80.8482)
+		(end 63.2222 80.8482)
 		(width 1)
 		(layer "F.Cu")
@@
 	)
 	(segment
-		(start 65.051 79.0194)
-		(end 58.2176 85.8528)
+		(start 67.564 80.7212)
+		(end 67.437 80.8482)
 		(width 1)
 		(layer "F.Cu")
@@
 		(start 68.5292 148.5265)
 		(end 55.4355 148.5265)
-		(width 0.2)
+		(width 0.8)
 		(layer "F.Cu")
 		(net 3)
@@
 		(start 55.4355 148.5265)
 		(end 53.6702 150.2918)
-		(width 0.2)
+		(width 0.8)
 		(layer "F.Cu")
 		(net 3)
@@
 		(start 68.8594 139.4333)
 		(end 53.9369 139.4333)
-		(width 0.2)
+		(width 0.8)
 		(layer "F.Cu")
 		(net 4)
@@
 		(start 68.8594 129.0955)
 		(end 54.2671 129.0955)
-		(width 0.2)
+		(width 0.8)
 		(layer "F.Cu")
 		(net 5)
 	)
 	(segment
-		(start 55.8419 118.7831)
-		(end 54.229 117.1702)
-		(width 0.2)
+		(start 62.3189 118.7831)
+		(end 60.706 117.1702)
+		(width 0.8)
 		(layer "F.Cu")
 		(net 6)
@@
 	(segment
 		(start 68.7578 118.7831)
-		(end 55.8419 118.7831)
-		(width 0.2)
+		(end 62.3189 118.7831)
+		(width 0.8)
+		(layer "F.Cu")
+		(net 6)
+	)
+	(segment
+		(start 60.706 117.1702)
+		(end 54.229 117.1702)
+		(width 0.8)
 		(layer "F.Cu")
 		(net 6)
@@
 		(start 93.0021 148.5265)
 		(end 71.0692 148.5265)
-		(width 0.2)
+		(width 0.8)
 		(layer "F.Cu")
 		(net 20)
@@
 		(start 100.0252 141.5034)
 		(end 93.0021 148.5265)
-		(width 0.2)
+		(width 0.8)
 		(layer "F.Cu")
 		(net 20)
@@
 		(start 97.1931 129.0955)
 		(end 71.3994 129.0955)
-		(width 0.2)
+		(width 0.8)
 		(layer "F.Cu")
 		(net 21)
@@
 		(start 100.0252 126.2634)
 		(end 97.1931 129.0955)
-		(width 0.2)
+		(width 0.8)
 		(layer "F.Cu")
 		(net 21)
@@
 		(start 100.0252 118.6434)
 		(end 71.4375 118.6434)
-		(width 0.2)
+		(width 0.8)
 		(layer "F.Cu")
 		(net 22)
@@
 		(start 76.9493 133.8834)
 		(end 71.3994 139.4333)
-		(width 0.2)
+		(width 0.8)
 		(layer "F.Cu")
 		(net 23)
@@
 		(start 100.0252 133.8834)
 		(end 76.9493 133.8834)
-		(width 0.2)
+		(width 0.8)
 		(layer "F.Cu")
 		(net 23)
@@
 		(start 85.5472 115.9764)
 		(end 70.2945 115.9764)
-		(width 0.2)
+		(width 0.8)
 		(layer "F.Cu")
 		(net 25)
@@
 		(start 73.0885 123.5964)
 		(end 70.1294 126.5555)
-		(width 0.2)
+		(width 0.8)
 		(layer "F.Cu")
 		(net 26)
@@
 		(start 85.598 123.5964)
 		(end 73.0885 123.5964)
-		(width 0.2)
+		(width 0.8)
 		(layer "F.Cu")
 		(net 26)
@@
 		(start 85.3694 131.3688)
 		(end 75.6539 131.3688)
-		(width 0.2)
+		(width 0.8)
 		(layer "F.Cu")
 		(net 27)
@@
 		(start 75.6539 131.3688)
 		(end 70.1294 136.8933)
-		(width 0.2)
+		(width 0.8)
 		(layer "F.Cu")
 		(net 27)
@@
 		(start 86.1314 138.9888)
 		(end 76.7969 138.9888)
-		(width 0.2)
+		(width 0.8)
 		(layer "F.Cu")
 		(net 28)
@@
 		(start 76.7969 138.9888)
 		(end 69.7992 145.9865)
-		(width 0.2)
+		(width 0.8)
 		(layer "F.Cu")
 		(net 28)
